Commit message: chganged sth

File: limo_description/urdf/limo_four_diff.xacro (robot description, xacro)
@@ -16,12 +16,12 @@
     <xacro:property name="wheel_length" value="0.045" />
     <xacro:property name="wheel_radius" value="0.045" />
-  <link name="base_footprint"/>
+  <link name="base_link"/>
   <joint name="base_joint" type="fixed">
-    <parent link="base_footprint"/>
-    <child link="base_link"/>
+    <parent link="base_link"/>
+    <child link="base_footprint"/>
     <origin xyz="0.0 0.0 0.15" rpy="0 0 0"/>
   </joint>
     <!-- Base link -->
-    <link name="base_link">
+    <link name="base_footprint">
         <visual>
             <origin xyz="0 0 -0.15" rpy="0 0 1.57" />
@@ -49,26 +49,26 @@
     <joint name="inertial_joint" type="fixed">
         <origin xyz="0 0 0" rpy="0 0 0" />
-        <parent link="base_link" />
+        <parent link="base_footprint" />
         <child link="inertial_link" />
     </joint>
-    <xacro:limo_laser parent_prefix="base_link" frame_prefix="laser">
+    <xacro:limo_laser parent_prefix="base_footprint" frame_prefix="laser">
         <origin xyz="0.103 0 -0.034" rpy="0 0 0"/>
     </xacro:limo_laser>
-    <xacro:limo_depth_camera parent_prefix="base_link" frame_prefix="depth_camera">
+    <xacro:limo_depth_camera parent_prefix="base_footprint" frame_prefix="depth_camera">
         <origin xyz="0.084 0 0.03" rpy="0 0 0"/>
     </xacro:limo_depth_camera>
-    <xacro:limo_imu parent_prefix="base_link" frame_prefix="imu">
+    <xacro:limo_imu parent_prefix="base_footprint" frame_prefix="imu">
         <origin xyz="0.0 0 -0.1" rpy="0 0 0"/>
     </xacro:limo_imu>
-    <xacro:limo_wheel parent_prefix="base_link" wheel_prefix="front_left" reflect="1">
+    <xacro:limo_wheel parent_prefix="base_footprint" wheel_prefix="front_left" reflect="1">
         <origin xyz="${wheelbase/2} ${track/2} ${wheel_vertical_offset}" rpy="0 0  0" />
     </xacro:limo_wheel>
-    <xacro:limo_wheel parent_prefix="base_link" wheel_prefix="front_right" reflect="-1">
+    <xacro:limo_wheel parent_prefix="base_footprint" wheel_prefix="front_right" reflect="-1">
         <origin xyz="${wheelbase/2} ${-track/2} ${wheel_vertical_offset}" rpy="${M_PI} 0 0" />
     </xacro:limo_wheel>
-    <xacro:limo_wheel parent_prefix="base_link" wheel_prefix="rear_left" reflect="1">
+    <xacro:limo_wheel parent_prefix="base_footprint" wheel_prefix="rear_left" reflect="1">
         <origin xyz="${-wheelbase/2} ${track/2} ${wheel_vertical_offset}" rpy="0 0 0" />
     </xacro:limo_wheel>
-    <xacro:limo_wheel parent_prefix="base_link" wheel_prefix="rear_right" reflect="-1">
+    <xacro:limo_wheel parent_prefix="base_footprint" wheel_prefix="rear_right" reflect="-1">
         <origin xyz="${-wheelbase/2} ${-track/2} ${wheel_vertical_offset}" rpy="${M_PI} 0 0" />
     </xacro:limo_wheel>

Commit message: added

File: limo_description/urdf/limo_four_diff.xacro (robot description, xacro)
@@ -16,12 +16,12 @@
     <xacro:property name="wheel_length" value="0.045" />
     <xacro:property name="wheel_radius" value="0.045" />
-  <link name="base_link"/>
+  <link name="base_footprint"/>
   <joint name="base_joint" type="fixed">
-    <parent link="base_link"/>
-    <child link="base_footprint"/>
+    <parent link="base_footprint"/>
+    <child link="base_link"/>
     <origin xyz="0.0 0.0 0.15" rpy="0 0 0"/>
   </joint>
     <!-- Base link -->
-    <link name="base_footprint">
+    <link name="base_link">
         <visual>
             <origin xyz="0 0 -0.15" rpy="0 0 1.57" />
@@ -49,26 +49,26 @@
     <joint name="inertial_joint" type="fixed">
         <origin xyz="0 0 0" rpy="0 0 0" />
-        <parent link="base_footprint" />
+        <parent link="base_link" />
         <child link="inertial_link" />
     </joint>
-    <xacro:limo_laser parent_prefix="base_footprint" frame_prefix="laser">
+    <xacro:limo_laser parent_prefix="base_link" frame_prefix="laser">
         <origin xyz="0.103 0 -0.034" rpy="0 0 0"/>
     </xacro:limo_laser>
-    <xacro:limo_depth_camera parent_prefix="base_footprint" frame_prefix="depth_camera">
+    <xacro:limo_depth_camera parent_prefix="base_link" frame_prefix="depth_camera">
         <origin xyz="0.084 0 0.03" rpy="0 0 0"/>
     </xacro:limo_depth_camera>
-    <xacro:limo_imu parent_prefix="base_footprint" frame_prefix="imu">
+    <xacro:limo_imu parent_prefix="base_link" frame_prefix="imu">
         <origin xyz="0.0 0 -0.1" rpy="0 0 0"/>
     </xacro:limo_imu>
-    <xacro:limo_wheel parent_prefix="base_footprint" wheel_prefix="front_left" reflect="1">
+    <xacro:limo_wheel parent_prefix="base_link" wheel_prefix="front_left" reflect="1">
         <origin xyz="${wheelbase/2} ${track/2} ${wheel_vertical_offset}" rpy="0 0  0" />
     </xacro:limo_wheel>
-    <xacro:limo_wheel parent_prefix="base_footprint" wheel_prefix="front_right" reflect="-1">
+    <xacro:limo_wheel parent_prefix="base_link" wheel_prefix="front_right" reflect="-1">
         <origin xyz="${wheelbase/2} ${-track/2} ${wheel_vertical_offset}" rpy="${M_PI} 0 0" />
     </xacro:limo_wheel>
-    <xacro:limo_wheel parent_prefix="base_footprint" wheel_prefix="rear_left" reflect="1">
+    <xacro:limo_wheel parent_prefix="base_link" wheel_prefix="rear_left" reflect="1">
         <origin xyz="${-wheelbase/2} ${track/2} ${wheel_vertical_offset}" rpy="0 0 0" />
     </xacro:limo_wheel>
-    <xacro:limo_wheel parent_prefix="base_footprint" wheel_prefix="rear_right" reflect="-1">
+    <xacro:limo_wheel parent_prefix="base_link" wheel_prefix="rear_right" reflect="-1">
         <origin xyz="${-wheelbase/2} ${-track/2} ${wheel_vertical_offset}" rpy="${M_PI} 0 0" />
     </xacro:limo_wheel>

Commit message: changed some params

File: limo_description/urdf/limo_four_diff.xacro (robot description, xacro)
@@ -20,5 +20,5 @@
     <parent link="base_footprint"/>
     <child link="base_link"/>
-    <origin xyz="0.0 0.0 0.15" rpy="0 0 0"/>
+    <origin xyz="0.0 0.0 0.5" rpy="0 0 0"/>
   </joint>
     <!-- Base link -->

Commit message: changed some params

File: limo_description/urdf/limo_four_diff.xacro (robot description, xacro)
@@ -20,5 +20,5 @@
     <parent link="base_footprint"/>
     <child link="base_link"/>
-    <origin xyz="0.0 0.0 0.5" rpy="0 0 0"/>
+    <origin xyz="0.0 0.0 0.15" rpy="0 0 0"/>
   </joint>
     <!-- Base link -->
